Commit message: Using one lidar instead of two

File: urdf/robot_assisted_cleaning_solution.gazebo.xacro (robot description, xacro)
@@ -16,5 +16,5 @@
 <!-- end  manual mode with teleop -->
 <!--#region laser-->
-  <gazebo reference="lidar_1">
+  <gazebo reference="lidar_top">
     <sensor type="ray" name="fullradious">
       <pose>0 0 0 0 0 0</pose>
@@ -24,14 +24,14 @@
         <scan>
           <horizontal>
-            <samples>720</samples>
-            <resolution>1</resolution>
-            <min_angle>-4.68</min_angle>
-            <max_angle>-0.03</max_angle>
+            <samples>400</samples>
+            <resolution>0.9</resolution>
+            <min_angle>0</min_angle>
+            <max_angle>6.283185</max_angle>
           </horizontal>
         </scan>
         <range>
-          <min>0.10</min>
-          <max>9.0</max>
-          <resolution>0.01</resolution>
+          <min>0.15</min>
+          <max>6.0</max>
+          <resolution>0.1</resolution>
         </range>
         <noise>
@@ -42,37 +42,6 @@
       </ray>
       <plugin name="gazebo_ros_head_hokuyo_controller" filename="libgazebo_ros_laser.so">
-        <topicName>scan1</topicName>
-        <frameName>lidar_1</frameName>
-      </plugin>
-    </sensor>
-  </gazebo>
-  <gazebo reference="lidar_2">
-    <sensor type="ray" name="halfradious">
-      <pose>0 0 0 0 0 0</pose>
-      <visualize>false</visualize>
-      <update_rate>40</update_rate>
-      <ray>
-        <scan>
-          <horizontal>
-            <samples>720</samples>
-            <resolution>1</resolution>
-            <min_angle>-1.54</min_angle>
-            <max_angle>3.11</max_angle>
-          </horizontal>
-        </scan>
-        <range>
-          <min>0.10</min>
-          <max>9.0</max>
-          <resolution>0.01</resolution>
-        </range>
-        <noise>
-          <type>gaussian</type>
-          <mean>0.0</mean>
-          <stddev>0.01</stddev>
-        </noise>
-      </ray>
-      <plugin name="gazebo_ros_head_hokuyo_controller" filename="libgazebo_ros_laser.so">
-        <topicName>scan2</topicName>
-        <frameName>lidar_2</frameName>
+        <topicName>scan</topicName>
+        <frameName>lidar_top</frameName>
       </plugin>
     </sensor>

File: urdf/robot_assisted_cleaning_solution.urdf.xacro (robot description, xacro)
@@ -372,4 +372,24 @@
       xyz="0 0 -1" />
   </joint>
+  <link name="lidar_top">
+    <visual>
+      <geometry>
+        <cylinder length="0.04080" radius="0.03785"/>
+      </geometry>
+    </visual>
+  </link>
+  <joint
+    name="lidar_top_joint"
+    type="fixed">
+    <origin
+      xyz="-0.00091 -0 0.1537"
+      rpy="0 0 0" />
+    <parent
+      link="base_link" />
+    <child
+      link="lidar_top" />
+    <axis
+      xyz="0 0 0" />
+  </joint>
   <link
     name="lidar_1">
